File: RC-KAKATA-CONTROL/JOYSTICK.kicad_sch (KiCad schematic)
At the start: 5 parts, among them U4 YK16S-L7.2-B10KA(32-8)-G-A29

Commit message: Completado el BOM
Parts:
- C40, C41, C42: LCSC Part (none) -> C14663
- R43: LCSC Part (none) -> C114065
Changed lines of the file:
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@@
+			)
+		)
+		(property "LCSC Part" "C14663"
+			(at 137.16 95.25 0)
+			(effects
+				(font
+					(size 1.27 1.27)
+				)
 			)
 		)
@@
 			)
 		)
+		(property "LCSC Part" "C14663"
+			(at 100.33 106.68 0)
+			(effects
+				(font
+					(size 1.27 1.27)
+				)
+			)
+		)
 		(pin "2"
 		)
@@
 			)
 		)
+		(property "LCSC Part" "C114065"
+			(at 137.16 77.47 0)
+			(effects
+				(font
+					(size 1.27 1.27)
+				)
+			)
+		)
 		(pin "1"
 		)
@@
 			)
 		)
+		(property "LCSC Part" "C14663"
+			(at 110.49 72.39 0)
+			(effects
+				(font
+					(size 1.27 1.27)
+				)
+			)
+		)
