File: RC-KAKATA-CONTROL/motor_driver.kicad_sch (KiCad schematic)
At the start: 2 parts, among them J2 Screw_Terminal_01x02

Commit message: Asignacion Ref. LCSC BOM
Asignacion de número de piezas de LCSC.
Queda pendiente cristal 25MHz y Power Supply.
Att.: Juan y Eric
Parts:
- J2: LCSC Part (none) -> C8465
- RC-VNH70-V1: now left out of the parts list
Changed lines of the file:
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@@
+			)
+		)
+		(property "LCSC Part" "C8465"
+			(at 187.96 107.95 0)
+			(effects
+				(font
+					(size 1.27 1.27)
+				)
+				(hide yes)
 			)
 		)
@@
 		(unit 1)
 		(exclude_from_sim no)
-		(in_bom yes)
+		(in_bom no)
 		(on_board yes)
 		(dnp no)
