File: RC-KAKATA-CONTROL/motor_driver.kicad_sch (KiCad schematic)
At the start: 2 parts, among them J2 Screw_Terminal_01x02

Commit message: Completado el BOM
Parts:
- J2: LCSC PN (none) -> C2915639; LCSC Part (none) -> C2915639
- RC-VNH70-V1: now not fitted
Changed lines of the file:
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@@
 		(on_board yes)
 		(dnp no)
-		(fields_autoplaced yes)
 		(property "Reference" "J2"
 			(at 190.5 107.9499 0)
@@
 			)
 		)
-		(property "LCSC PN" ""
-			(at 187.96 107.95 0)
-			(effects
-				(font
-					(size 1.27 1.27)
-				)
-				(hide yes)
+		(property "LCSC PN" "C2915639"
+			(at 187.96 107.95 0)
+			(effects
+				(font
+					(size 1.27 1.27)
+				)
+				(hide yes)
+			)
+		)
+		(property "PART_NUMBER" ""
+			(at 187.96 107.95 0)
+			(effects
+				(font
+					(size 1.27 1.27)
+				)
+				(hide yes)
+			)
+		)
+		(property "LCSC Part #" ""
+			(at 187.96 107.95 0)
+			(effects
+				(font
+					(size 1.27 1.27)
+				)
+				(hide yes)
+			)
+		)
+		(property "LCSC Part" "C2915639"
+			(at 188.214 105.41 0)
+			(effects
+				(font
+					(size 1.27 1.27)
+				)
 			)
 		)
@@
 		)
 		(instances
-			(project "RC-KAKATA-CONTROL"
+			(project ""
+				(path "/739b16ea-69b1-41ec-be07-897a0cbc3062"
+					(reference "J9")
+					(unit 1)
+				)
 				(path "/739b16ea-69b1-41ec-be07-897a0cbc3062/2de8daa4-f828-4eee-a9c1-fedae33e84fa"
 					(reference "J9")
@@
 		(in_bom yes)
 		(on_board yes)
-		(dnp no)
+		(dnp yes)
 		(property "Reference" "RC-VNH70-V1"
 			(at 140.0967 92.71 0)
