File: RC-KAKATA-CONTROL/power_supply.kicad_sch (KiCad schematic)
At the start: 49 parts, among them J3 Screw_Terminal_01x02, J4 Screw_Terminal_01x02, U1 PS-TO220, U2 PS-TO220

Commit message: Asignacion Ref. LCSC BOM
Asignacion de número de piezas de LCSC.
Queda pendiente cristal 25MHz y Power Supply.
Att.: Juan y Eric
Parts:
- C1, C10, C11, C12, C13, C14, C16, C17, C18, C2, C21, C25, C3, C4, C5, C6, C7, C8, C9: LCSC Part (none) -> C109474
- C20, C22: LCSC Part (none) -> C106248
- C23: LCSC Part (none) -> C33129640
- C45, C47, C48, C49: LCSC Part (none) -> C2887276
- D1, D3: LCSC Part (none) -> C22452
- D2: LCSC Part (none) -> C193402
- D4, D6: LCSC Part (none) -> C19077515
- D5: LCSC Part (none) -> C2649858
- J3, J4: LCSC Part (none) -> C8465
- L1: LCSC Part (none) -> C701178
- LED1, LED2, LED3, LED4: LCSC Part (none) -> C19171390
- R10, R9: LCSC Part (none) -> C114662
- R11, R6, R8: LCSC Part (none) -> C22548
- R12: LCSC Part (none) -> C705763
- R5, R7: LCSC Part (none) -> C95204
