File: RC-KAKATA-CONTROL/rf_in.kicad_sch (KiCad schematic)
At the start: 2 parts

Commit message: Asignacion Ref. LCSC BOM
Asignacion de número de piezas de LCSC.
Queda pendiente cristal 25MHz y Power Supply.
Att.: Juan y Eric
Parts:
- RF1: now left out of the parts list
Changed lines of the file:
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@@
 		(unit 1)
 		(exclude_from_sim no)
-		(in_bom yes)
+		(in_bom no)
 		(on_board yes)
 		(dnp no)
