File: RC-KAKATA-CONTROL/rf_in.kicad_sch (KiCad schematic)
At the start: 2 parts

Commit message: Completado el BOM
Parts:
- JP3: LCSC Part (none) -> C52016391
- RF1: now not fitted
Changed lines of the file:
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@@
 		(in_bom yes)
 		(on_board yes)
-		(dnp no)
+		(dnp yes)
 		(fields_autoplaced yes)
 		(property "Reference" "RF1"
@@
 			)
 		)
+		(property "LCSC Part" "C52016391"
+			(at 93.98 121.92 90)
+			(effects
+				(font
+					(size 1.27 1.27)
+				)
+			)
+		)

Commit message: V1.0 Enviada a fabricar
Parts:
- JP3: now in the parts list
Changed lines of the file:
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@@
 		(unit 1)
 		(exclude_from_sim no)
-		(in_bom no)
+		(in_bom yes)
 		(on_board yes)
 		(dnp no)
-		(fields_autoplaced yes)
 		(property "Reference" "JP3"
 			(at 91.44 120.6499 90)
@@
 		)
 		(property "LCSC Part" "C52016391"
-			(at 93.98 121.92 90)
+			(at 101.6 124.46 90)
 			(effects
 				(font
+					(size 1.27 1.27)
+				)
+			)
+		)
+		(property "PART_NUMBER" ""
+			(at 93.98 121.92 0)
+			(effects
+				(font
+					(size 1.27 1.27)
+				)
+				(hide yes)
+			)
+		)
+		(property "LCSC Part #" ""
+			(at 93.98 121.92 0)
+			(effects
+				(font
+					(size 1.27 1.27)
+				)
+				(hide yes)
+			)
+		)
+		(property "Manufacturer" ""
+			(at 93.98 121.92 0)
+			(effects
+				(font
+					(size 1.27 1.27)
+				)
+				(hide yes)
+			)
+		)
+		(property "VOL" ""
+			(at 93.98 121.92 0)
+			(effects
+				(font
+					(size 1.27 1.27)
+				)
+			)
+		)
+		(property "TOL" ""
+			(at 93.98 121.92 0)
+			(effects
+				(font
