File: RC-KAKATA-CONTROL/RC-KAKATA-CONTROL.kicad_pcb (KiCad board)
At the start: 6 copper layers, 160 x 160 mm, 182 parts, among them J1 Conn_02x20_Socket_DG250T-5.0-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, J10 DB125-2.54-4P-GN, J11 Screw_Terminal_01x02, J12 Conn_01x07, J13 Screw_Terminal_01x02, J14 DB125-2.54-4P-GN, J17 Screw_Terminal_01x02, J19 Screw_Terminal_01x02, J2 Screw_Terminal_01x02, J21 Screw_Terminal_01x02, J23 Screw_Terminal_01x02, J25 Conn_02x20_Socket_DG250T-5.0-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, J3 Screw_Terminal_01x02, J4 Screw_Terminal_01x02, J5 Screw_Terminal_01x02, J6 Raspberry_Pi_2x20_PTH, J7 Screw_Terminal_01x02, J8 DB125-2.54-4P-GN, J9 Screw_Terminal_01x02, SW1 TS-1088-AR02016, SW2 TS-1088-AR02016, SW3 TS-1088-AR02016, SW4 TS-1088-AR02016, SW6 TS-1088-AR02016, U1 PS-TO220, U13 ICM-20689, U2 PS-TO220, U3 STM32H743IIT6, U4 YK16S-L7.2-B10KA(32-8)-G-A29, U8 W25Q128JVSIQTR, X1 SMD3225-4, X2 Q13MC3061000300

Commit message: V1.0 Enviada a fabricar
Parts:
- removed C27: 100NF, 4ms_Capacitor:C_0603
- removed C28: 10NF, 4ms_Capacitor:C_0603
- removed C44: 2.2uF, 4ms_Capacitor:C_0603
- removed C46: 0.47uF, 4ms_Capacitor:C_0603
- removed U13: ICM-20689, EasyEDA:QFN-24_L4.0-W4.0-P0.50-TL-EP2.6
- added C15: 10nF, Capacitor_SMD_AKL:C_0603_1608Metric, F.Cu at (171.6, 171.6)
- added C55: 100nF, Capacitor_SMD_AKL:C_0603_1608Metric, F.Cu at (176.7, 171.6)
- added C56: 100nF, Capacitor_SMD_AKL:C_0603_1608Metric, F.Cu at (177.8, 169.5)
- added C57: 100nF, Capacitor_SMD_AKL:C_0603_1608Metric, F.Cu at (175.3, 164.3)
- added U5: MPU-6050_C24112, EasyEDA:QFN-24_L4.0-W4.0-P0.50-BL-EP2.7, F.Cu at (173.4, 168.2)
- C36, C37: value 8pF -> 16pF
- C38, C39: value 12pF -> 20pF
- R1, R2, R3, R4: value 10K -> 4.7K
- R17, R45, R53, R54, R55: value 10K -> 22K
- U8: value W25Q128JVSIQTR -> W25Q128JVSIQ
- X1: value SMD3225-4 -> 25MHZ
- X2: value Q13MC3061000300 -> 32.768kHz
Routing:
- net /RF_DATA_UART_TX: track 52.5 -> 44.4 mm
- net GND: track 220.5 -> 227.5 mm, vias 1694 -> 1693
- net /ACC_GYR_INT: track 57.8 -> 62.1 mm
- net Net-(U5-REGOUT): track 0.00 -> 3.32 mm
- net /ACC_GYR_SDA: track 39.5 -> 42.8 mm
- net /ACC_GYR_SCL: track 48.0 -> 50.6 mm
- net Net-(JP2-C): track 18.8 -> 21.1 mm, vias 0 -> 1
- net +3.3V: track 174.8 -> 172.6 mm
- net Net-(U13-REGOUT): track 2.10 -> 0.00 mm
- net Net-(U5-CPOUT): track 0.00 -> 2.08 mm
- net /RF_DATA_TIMER: track 75.2 -> 74.4 mm
